File: rear/electronics/bikepixel rear/bikepixel rear.sch (KiCad schematic (older format))
At the start: 14 parts, among them J1 Power, J2 Arduino, J3 Matrix, SW0 on/off, SW1 mode, SW2 color, SW3 effect

Commit message: Added files for bike pixel rear with battery support and 3d printed case
Other:
- moved on the sheet: R3, R4, R5
Changed lines of the file:
@@
 L bikepxiel~rear:SW_Push_Dual_Vertical SW1
 U 1 1 60777A1F
-P 5100 4900
-F 0 "SW1" H 5100 5190 50  0000 C CNN
-F 1 "mode" H 5100 5099 50  0000 C CNN
-F 2 "Button_Switch_THT:SW_Tactile_SPST_Angled_PTS645Vx58-2LFS" H 5550 5200 50  0001 C CNN
-F 3 "" H 5550 5200 50  0001 C CNN
-	1    5100 4900
+P 5100 4600
+F 0 "SW1" H 5100 4890 50  0000 C CNN
+F 1 "mode" H 5100 4799 50  0000 C CNN
+F 2 "Button_Switch_THT:SW_Tactile_SPST_Angled_PTS645Vx58-2LFS" H 5550 4900 50  0001 C CNN
+F 3 "" H 5550 4900 50  0001 C CNN
+	1    5100 4600
 	1    0    0    -1
 $EndComp
@@
 L bikepxiel~rear:SW_Push_Dual_Vertical SW2
 U 1 1 6077975F
-P 5850 4900
-F 0 "SW2" H 5850 5190 50  0000 C CNN
-F 1 "color" H 5850 5099 50  0000 C CNN
-F 2 "Button_Switch_THT:SW_Tactile_SPST_Angled_PTS645Vx58-2LFS" H 6300 5200 50  0001 C CNN
-F 3 "" H 6300 5200 50  0001 C CNN
-	1    5850 4900
+P 5850 4600
+F 0 "SW2" H 5850 4890 50  0000 C CNN
+F 1 "color" H 5850 4799 50  0000 C CNN
+F 2 "Button_Switch_THT:SW_Tactile_SPST_Angled_PTS645Vx58-2LFS" H 6300 4900 50  0001 C CNN
+F 3 "" H 6300 4900 50  0001 C CNN
+	1    5850 4600
 	1    0    0    -1
 $EndComp
@@
 L bikepxiel~rear:SW_Push_Dual_Vertical SW3
 U 1 1 6077AEBC
-P 6600 4900
-F 0 "SW3" H 6600 5190 50  0000 C CNN
-F 1 "effect" H 6600 5099 50  0000 C CNN
-F 2 "Button_Switch_THT:SW_Tactile_SPST_Angled_PTS645Vx58-2LFS" H 7050 5200 50  0001 C CNN
-F 3 "" H 7050 5200 50  0001 C CNN
-	1    6600 4900
+P 6600 4600
+F 0 "SW3" H 6600 4890 50  0000 C CNN
+F 1 "effect" H 6600 4799 50  0000 C CNN
+F 2 "Button_Switch_THT:SW_Tactile_SPST_Angled_PTS645Vx58-2LFS" H 7050 4900 50  0001 C CNN
+F 3 "" H 7050 4900 50  0001 C CNN
+	1    6600 4600
 	1    0    0    -1
 $EndComp
@@
 L Device:R R3
 U 1 1 60783D96
-P 5400 4200
-F 0 "R3" V 5500 4250 50  0000 C CNN
-F 1 "10k" V 5400 4200 50  0000 C CNN
-F 2 "Resistor_THT:R_Axial_DIN0207_L6.3mm_D2.5mm_P7.62mm_Horizontal" V 5330 4200 50  0001 C CNN
-F 3 "~" H 5400 4200 50  0001 C CNN
-	1    5400 4200
+P 5400 4350
+F 0 "R3" V 5500 4400 50  0000 C CNN
+F 1 "10k" V 5400 4350 50  0000 C CNN
+F 2 "Resistor_THT:R_Axial_DIN0207_L6.3mm_D2.5mm_P7.62mm_Horizontal" V 5330 4350 50  0001 C CNN
+F 3 "~" H 5400 4350 50  0001 C CNN
+	1    5400 4350
 	1    0    0    -1
 $EndComp
@@
 L Device:R R5
 U 1 1 607846D3
-P 6900 4200
-F 0 "R5" V 7000 4250 50  0000 C CNN
-F 1 "10k" V 6900 4200 50  0000 C CNN
-F 2 "Resistor_THT:R_Axial_DIN0207_L6.3mm_D2.5mm_P7.62mm_Horizontal" V 6830 4200 50  0001 C CNN
-F 3 "~" H 6900 4200 50  0001 C CNN
-	1    6900 4200
+P 6900 4350
+F 0 "R5" V 7000 4400 50  0000 C CNN
+F 1 "10k" V 6900 4350 50  0000 C CNN
+F 2 "Resistor_THT:R_Axial_DIN0207_L6.3mm_D2.5mm_P7.62mm_Horizontal" V 6830 4350 50  0001 C CNN
+F 3 "~" H 6900 4350 50  0001 C CNN
+	1    6900 4350
 	1    0    0    -1
 $EndComp
@@
 L Device:R R4
 U 1 1 60784939
-P 6100 4200
-F 0 "R4" V 6050 4350 50  0000 C CNN
-F 1 "10k" V 6100 4200 50  0000 C CNN
-F 2 "Resistor_THT:R_Axial_DIN0207_L6.3mm_D2.5mm_P7.62mm_Horizontal" V 6030 4200 50  0001 C CNN
-F 3 "~" H 6100 4200 50  0001 C CNN
-	1    6100 4200
+P 6100 4350
+F 0 "R4" V 6050 4500 50  0000 C CNN
+F 1 "10k" V 6100 4350 50  0000 C CNN
+F 2 "Resistor_THT:R_Axial_DIN0207_L6.3mm_D2.5mm_P7.62mm_Horizontal" V 6030 4350 50  0001 C CNN
+F 3 "~" H 6100 4350 50  0001 C CNN
+	1    6100 4350
 	1    0    0    -1
 $EndComp
@@
 	1    0    0    -1
 $EndComp
-$Comp
-L power:GND #PWR0102
-U 1 1 60791BDB
-P 4800 5150
-F 0 "#PWR0102" H 4800 4900 50  0001 C CNN
-F 1 "GND" H 4805 4977 50  0000 C CNN
-F 2 "" H 4800 5150 50  0001 C CNN
-F 3 "" H 4800 5150 50  0001 C CNN
-	1    4800 5150
-	1    0    0    -1
-$EndComp
-$Comp
-L power:GND #PWR0103
-U 1 1 60792893
-P 5550 5150
-F 0 "#PWR0103" H 5550 4900 50  0001 C CNN
-F 1 "GND" H 5555 4977 50  0000 C CNN
-F 2 "" H 5550 5150 50  0001 C CNN
-F 3 "" H 5550 5150 50  0001 C CNN
-	1    5550 5150
-	1    0    0    -1
-$EndComp
-$Comp
-L power:GND #PWR0104
-U 1 1 60792EB2
-P 6300 5150
-F 0 "#PWR0104" H 6300 4900 50  0001 C CNN
-F 1 "GND" H 6305 4977 50  0000 C CNN
-F 2 "" H 6300 5150 50  0001 C CNN
-F 3 "" H 6300 5150 50  0001 C CNN
-	1    6300 5150
-	1    0    0    -1
-$EndComp
-Wire Wire Line
-	4900 4900 4800 4900
-Wire Wire Line
-	4800 4900 4800 5150
-Wire Wire Line
-	5400 4900 5300 4900
+Wire Wire Line
+	4900 4600 4800 4600
+Wire Wire Line
+	5400 4600 5300 4600
 $Comp
 L power:+5V #PWR0105
@@
 	0    1    1    0
 $EndComp
-$Comp
-L power:+5V #PWR0108
-U 1 1 607AFAF7
-P 5400 4000
-F 0 "#PWR0108" H 5400 3850 50  0001 C CNN
-F 1 "+5V" H 5300 4100 50  0000 C CNN
-F 2 "" H 5400 4000 50  0001 C CNN
-F 3 "" H 5400 4000 50  0001 C CNN
-	1    5400 4000
-	1    0    0    -1
-$EndComp
-$Comp
-L power:+5V #PWR0109
-U 1 1 607B193C
-P 6100 4000
-F 0 "#PWR0109" H 6100 3850 50  0001 C CNN
-F 1 "+5V" H 6100 4150 50  0000 C CNN
-F 2 "" H 6100 4000 50  0001 C CNN
-F 3 "" H 6100 4000 50  0001 C CNN
-	1    6100 4000
-	1    0    0    -1
-$EndComp
-$Comp
-L power:+5V #PWR0110
-U 1 1 607B24A4
-P 6900 4000
-F 0 "#PWR0110" H 6900 3850 50  0001 C CNN
-F 1 "+5V" H 6800 4100 50  0000 C CNN
-F 2 "" H 6900 4000 50  0001 C CNN
-F 3 "" H 6900 4000 50  0001 C CNN
-	1    6900 4000
-	1    0    0    -1
-$EndComp
-Wire Wire Line
-	6900 4900 6800 4900
-Wire Wire Line
-	6300 5150 6300 4900
-Wire Wire Line
-	6300 4900 6400 4900
-Wire Wire Line
-	5550 5150 5550 4900
-Wire Wire Line
-	5550 4900 5650 4900
+Wire Wire Line
+	6900 4600 6800 4600
+Wire Wire Line
+	6300 4850 6300 4600
+Wire Wire Line
+	6300 4600 6400 4600
+Wire Wire Line
+	5550 4850 5550 4600
+Wire Wire Line
+	5550 4600 5650 4600
 $Comp
 L Connector:Conn_01x07_Female J2
@@
 $EndComp
 Wire Wire Line
-	6900 4350 6900 4450
-Wire Wire Line
-	5400 4350 5400 4450
-Wire Wire Line
-	6400 3150 6400 4450
-Wire Wire Line
-	6400 4450 6900 4450
-Connection ~ 6900 4450
-Wire Wire Line
-	6900 4450 6900 4900
-Wire Wire Line
-	5400 4450 6000 4450
-Wire Wire Line
-	6000 4450 6000 3150
-Connection ~ 5400 4450
-Wire Wire Line
-	5400 4450 5400 4900
+	6400 4150 6900 4150
 $Comp
 L Connector:Conn_01x03_Female J1
@@
 Connection ~ 5000 3200
 Wire Wire Line
-	5400 4050 5400 4000
-Wire Wire Line
-	6900 4050 6900 4000
-Wire Wire Line
 	5550 3550 5650 3550
 Wire Wire Line
@@
 Note that in the matrix specs a 1000 uF \ncapacitator is recommended but due to \nsize restrctions a smaller one is used.
 Wire Wire Line
-	6100 4000 6100 4050
-Wire Wire Line
-	6100 4350 6100 4450
-Wire Wire Line
-	6100 4900 6050 4900
-Wire Wire Line
-	6100 4450 6200 4450
-Wire Wire Line
-	6200 3150 6200 4450
-Connection ~ 6100 4450
-Wire Wire Line
-	6100 4450 6100 4900
-$Comp
-L power:GND #PWR?
+	6100 4600 6050 4600
+Wire Wire Line
+	6100 4150 6200 4150
+$Comp
+L power:GND #PWR0102
 U 1 1 60C2CA88
 P 6300 3450
-F 0 "#PWR?" H 6300 3200 50  0001 C CNN
+F 0 "#PWR0102" H 6300 3200 50  0001 C CNN
 F 1 "GND" H 6305 3277 50  0000 C CNN
 F 2 "" H 6300 3450 50  0001 C CNN
@@
 Wire Wire Line
 	6500 3200 6500 3150
+Wire Wire Line
+	4800 4600 4800 4850
+$Comp
+L power:GND #PWR0103
+U 1 1 616EFCE1
+P 5400 4050
+F 0 "#PWR0103" H 5400 3800 50  0001 C CNN
+F 1 "GND" H 5400 3900 50  0000 C CNN
+F 2 "" H 5400 4050 50  0001 C CNN
+F 3 "" H 5400 4050 50  0001 C CNN
+	1    5400 4050
+	-1   0    0    1
+$EndComp
+$Comp
+L power:GND #PWR0104
+U 1 1 616F03D4
+P 6100 4050
+F 0 "#PWR0104" H 6100 3800 50  0001 C CNN
+F 1 "GND" H 6100 3900 50  0000 C CNN
+F 2 "" H 6100 4050 50  0001 C CNN
+F 3 "" H 6100 4050 50  0001 C CNN
+	1    6100 4050
+	-1   0    0    1
+$EndComp
+$Comp
+L power:GND #PWR0108
+U 1 1 616F0AF2
+P 6900 4050
+F 0 "#PWR0108" H 6900 3800 50  0001 C CNN
+F 1 "GND" H 6900 3900 50  0000 C CNN
+F 2 "" H 6900 4050 50  0001 C CNN
+F 3 "" H 6900 4050 50  0001 C CNN
+	1    6900 4050
+	-1   0    0    1
+$EndComp
+$Comp
+L power:+5V #PWR0109
+U 1 1 616F248F
+P 4800 4850
+F 0 "#PWR0109" H 4800 4700 50  0001 C CNN
+F 1 "+5V" H 4815 5023 50  0000 C CNN
+F 2 "" H 4800 4850 50  0001 C CNN
+F 3 "" H 4800 4850 50  0001 C CNN
+	1    4800 4850
+	-1   0    0    1
+$EndComp
+$Comp
+L power:+5V #PWR0110
+U 1 1 616F30CA
+P 5550 4850
+F 0 "#PWR0110" H 5550 4700 50  0001 C CNN
+F 1 "+5V" H 5565 5023 50  0000 C CNN
+F 2 "" H 5550 4850 50  0001 C CNN
+F 3 "" H 5550 4850 50  0001 C CNN
+	1    5550 4850
+	-1   0    0    1
+$EndComp
+$Comp
+L power:+5V #PWR0111
+U 1 1 616F3611
+P 6300 4850
+F 0 "#PWR0111" H 6300 4700 50  0001 C CNN
+F 1 "+5V" H 6315 5023 50  0000 C CNN
+F 2 "" H 6300 4850 50  0001 C CNN
+F 3 "" H 6300 4850 50  0001 C CNN
+	1    6300 4850
+	-1   0    0    1
+$EndComp
+Wire Wire Line
+	5400 4600 5400 4500
+Wire Wire Line
+	6000 4150 5400 4150
+Wire Wire Line
+	5400 4150 5400 4200
+Wire Wire Line
+	6100 4200 6100 4150
+Wire Wire Line
+	6100 4500 6100 4600
+Wire Wire Line
+	6000 3150 6000 4150
+Wire Wire Line
+	6100 4150 6100 4050
+Connection ~ 6100 4150
+Wire Wire Line
+	6200 4150 6200 3150
+Wire Wire Line
+	6900 4600 6900 4500
+Wire Wire Line
+	6900 4200 6900 4150
+Connection ~ 6900 4150
+Wire Wire Line
+	6900 4150 6900 4050
+Wire Wire Line
+	6400 4150 6400 3150
+Wire Wire Line
+	5400 4150 5400 4050
+Connection ~ 5400 4150
 $EndSCHEMATC

Commit message: Added PCB design. Improved documentation
Parts:
- removed SW1: mode, Button_Switch_THT:SW_Tactile_SPST_Angled_PTS645Vx58-2LFS, symbol bikepxiel~rear:SW_Push_Dual_Vertical
- removed SW2: color, Button_Switch_THT:SW_Tactile_SPST_Angled_PTS645Vx58-2LFS, symbol bikepxiel~rear:SW_Push_Dual_Vertical
- removed SW3: effect, Button_Switch_THT:SW_Tactile_SPST_Angled_PTS645Vx58-2LFS, symbol bikepxiel~rear:SW_Push_Dual_Vertical
- added SW1: mode, Button_Switch_THT:SW_Tactile_SPST_Angled_PTS645Vx58-2LFS, symbol bikepxiel~rear:SW_Push
- added SW2: color, Button_Switch_THT:SW_Tactile_SPST_Angled_PTS645Vx58-2LFS, symbol bikepxiel~rear:SW_Push
- added SW3: effect, Button_Switch_THT:SW_Tactile_SPST_Angled_PTS645Vx58-2LFS, symbol bikepxiel~rear:SW_Push
Other:
- moved on the sheet: R3, R4, R5
Changed lines of the file:
@@
 $EndDescr
-$Comp
-L bikepxiel~rear:SW_Push_Dual_Vertical SW1
-U 1 1 60777A1F
-P 5100 4600
-F 0 "SW1" H 5100 4890 50  0000 C CNN
-F 1 "mode" H 5100 4799 50  0000 C CNN
-F 2 "Button_Switch_THT:SW_Tactile_SPST_Angled_PTS645Vx58-2LFS" H 5550 4900 50  0001 C CNN
-F 3 "" H 5550 4900 50  0001 C CNN
-	1    5100 4600
-	1    0    0    -1
-$EndComp
-$Comp
-L bikepxiel~rear:SW_Push_Dual_Vertical SW2
-U 1 1 6077975F
-P 5850 4600
-F 0 "SW2" H 5850 4890 50  0000 C CNN
-F 1 "color" H 5850 4799 50  0000 C CNN
-F 2 "Button_Switch_THT:SW_Tactile_SPST_Angled_PTS645Vx58-2LFS" H 6300 4900 50  0001 C CNN
-F 3 "" H 6300 4900 50  0001 C CNN
-	1    5850 4600
-	1    0    0    -1
-$EndComp
-$Comp
-L bikepxiel~rear:SW_Push_Dual_Vertical SW3
-U 1 1 6077AEBC
-P 6600 4600
-F 0 "SW3" H 6600 4890 50  0000 C CNN
-F 1 "effect" H 6600 4799 50  0000 C CNN
-F 2 "Button_Switch_THT:SW_Tactile_SPST_Angled_PTS645Vx58-2LFS" H 7050 4900 50  0001 C CNN
-F 3 "" H 7050 4900 50  0001 C CNN
-	1    6600 4600
-	1    0    0    -1
-$EndComp
 $Comp
 L Device:R R2
@@
 $EndComp
 $Comp
-L Device:R R3
-U 1 1 60783D96
-P 5400 4350
-F 0 "R3" V 5500 4400 50  0000 C CNN
-F 1 "10k" V 5400 4350 50  0000 C CNN
-F 2 "Resistor_THT:R_Axial_DIN0207_L6.3mm_D2.5mm_P7.62mm_Horizontal" V 5330 4350 50  0001 C CNN
-F 3 "~" H 5400 4350 50  0001 C CNN
-	1    5400 4350
-	1    0    0    -1
-$EndComp
-$Comp
 L Device:R R6
 U 1 1 60783FAA
@@
 $EndComp
 $Comp
-L Device:R R5
-U 1 1 607846D3
-P 6900 4350
-F 0 "R5" V 7000 4400 50  0000 C CNN
-F 1 "10k" V 6900 4350 50  0000 C CNN
-F 2 "Resistor_THT:R_Axial_DIN0207_L6.3mm_D2.5mm_P7.62mm_Horizontal" V 6830 4350 50  0001 C CNN
-F 3 "~" H 6900 4350 50  0001 C CNN
-	1    6900 4350
-	1    0    0    -1
-$EndComp
-$Comp
-L Device:R R4
-U 1 1 60784939
-P 6100 4350
-F 0 "R4" V 6050 4500 50  0000 C CNN
-F 1 "10k" V 6100 4350 50  0000 C CNN
-F 2 "Resistor_THT:R_Axial_DIN0207_L6.3mm_D2.5mm_P7.62mm_Horizontal" V 6030 4350 50  0001 C CNN
-F 3 "~" H 6100 4350 50  0001 C CNN
-	1    6100 4350
-	1    0    0    -1
-$EndComp
-$Comp
 L power:GND #PWR0101
 U 1 1 6078E32E
@@
 	1    0    0    -1
 $EndComp
-Wire Wire Line
-	4900 4600 4800 4600
-Wire Wire Line
-	5400 4600 5300 4600
 $Comp
 L power:+5V #PWR0105
@@
 	0    1    1    0
 $EndComp
-Wire Wire Line
-	6900 4600 6800 4600
-Wire Wire Line
-	6300 4850 6300 4600
-Wire Wire Line
-	6300 4600 6400 4600
-Wire Wire Line
-	5550 4850 5550 4600
-Wire Wire Line
-	5550 4600 5650 4600
 $Comp
 L Connector:Conn_01x07_Female J2
@@
 	0    -1   -1   0
 $EndComp
-Wire Wire Line
-	6400 4150 6900 4150
 $Comp
 L Connector:Conn_01x03_Female J1
@@
 Text Notes 8000 3150 0    39   ~ 0
 Note that in the matrix specs a 1000 uF \ncapacitator is recommended but due to \nsize restrctions a smaller one is used.
-Wire Wire Line
-	6100 4600 6050 4600
-Wire Wire Line
-	6100 4150 6200 4150
 $Comp
 L power:GND #PWR0102
@@
 	6500 3200 6500 3150
 Wire Wire Line
-	4800 4600 4800 4850
-$Comp
-L power:GND #PWR0103
-U 1 1 616EFCE1
+	6100 4900 6050 4900
+Wire Wire Line
+	5550 4900 5650 4900
+Wire Wire Line
+	6300 4900 6400 4900
+Wire Wire Line
+	5400 4900 5300 4900
+Wire Wire Line
+	4900 4900 4800 4900
+$Comp
+L Device:R R4
+U 1 1 60784939
+P 6100 4250
+F 0 "R4" V 6050 4400 50  0000 C CNN
+F 1 "10k" V 6100 4250 50  0000 C CNN
+F 2 "Resistor_THT:R_Axial_DIN0207_L6.3mm_D2.5mm_P7.62mm_Horizontal" V 6030 4250 50  0001 C CNN
+F 3 "~" H 6100 4250 50  0001 C CNN
+	1    6100 4250
+	1    0    0    -1
+$EndComp
+$Comp
+L Device:R R5
+U 1 1 607846D3
+P 6900 4250
+F 0 "R5" V 7000 4300 50  0000 C CNN
+F 1 "10k" V 6900 4250 50  0000 C CNN
+F 2 "Resistor_THT:R_Axial_DIN0207_L6.3mm_D2.5mm_P7.62mm_Horizontal" V 6830 4250 50  0001 C CNN
+F 3 "~" H 6900 4250 50  0001 C CNN
+	1    6900 4250
+	1    0    0    -1
+$EndComp
+$Comp
+L Device:R R3
+U 1 1 60783D96
+P 5400 4250
+F 0 "R3" V 5500 4300 50  0000 C CNN
+F 1 "10k" V 5400 4250 50  0000 C CNN
+F 2 "Resistor_THT:R_Axial_DIN0207_L6.3mm_D2.5mm_P7.62mm_Horizontal" V 5330 4250 50  0001 C CNN
+F 3 "~" H 5400 4250 50  0001 C CNN
+	1    5400 4250
+	1    0    0    -1
+$EndComp
+Wire Wire Line
+	5400 4050 5400 4100
+Wire Wire Line
+	6100 4050 6100 4100
+Wire Wire Line
+	6900 4050 6900 4100
+Wire Wire Line
+	5400 4900 5400 4500
+Wire Wire Line
+	6100 4900 6100 4500
+Wire Wire Line
+	6900 4900 6900 4500
+Wire Wire Line
+	5400 4500 6000 4500
+Wire Wire Line
+	6000 3150 6000 4500
+Connection ~ 5400 4500
+Wire Wire Line
+	5400 4500 5400 4400
+Wire Wire Line
+	6100 4500 6200 4500
+Wire Wire Line
+	6200 3150 6200 4500
+Connection ~ 6100 4500
+Wire Wire Line
+	6100 4500 6100 4400
+Wire Wire Line
+	6900 4500 6400 4500
+Wire Wire Line
+	6400 3150 6400 4500
+Connection ~ 6900 4500
+Wire Wire Line
+	6900 4500 6900 4400
+$Comp
+L bikepxiel~rear:SW_Push SW1
+U 1 1 61A73CDC
+P 5100 4900
+F 0 "SW1" H 5100 5185 50  0000 C CNN
+F 1 "mode" H 5100 5094 50  0000 C CNN
+F 2 "Button_Switch_THT:SW_Tactile_SPST_Angled_PTS645Vx58-2LFS" H 5100 5100 50  0001 C CNN
+F 3 "" H 5100 5100 50  0001 C CNN
+	1    5100 4900
+	1    0    0    -1
+$EndComp
+$Comp
+L bikepxiel~rear:SW_Push SW2
+U 1 1 61A78EBE
+P 5850 4900
+F 0 "SW2" H 5850 5185 50  0000 C CNN
+F 1 "color" H 5850 5094 50  0000 C CNN
+F 2 "Button_Switch_THT:SW_Tactile_SPST_Angled_PTS645Vx58-2LFS" H 5850 5100 50  0001 C CNN
+F 3 "" H 5850 5100 50  0001 C CNN
+	1    5850 4900
+	1    0    0    -1
+$EndComp
+$Comp
+L bikepxiel~rear:SW_Push SW3
+U 1 1 61A799E7
+P 6600 4900
+F 0 "SW3" H 6600 5185 50  0000 C CNN
+F 1 "effect" H 6600 5094 50  0000 C CNN
+F 2 "Button_Switch_THT:SW_Tactile_SPST_Angled_PTS645Vx58-2LFS" H 6600 5100 50  0001 C CNN
+F 3 "" H 6600 5100 50  0001 C CNN
+	1    6600 4900
+	1    0    0    -1
+$EndComp
+Wire Wire Line
+	6900 4900 6800 4900
+$Comp
+L power:+5V #PWR0103
+U 1 1 61A81449
 P 5400 4050
-F 0 "#PWR0103" H 5400 3800 50  0001 C CNN
-F 1 "GND" H 5400 3900 50  0000 C CNN
+F 0 "#PWR0103" H 5400 3900 50  0001 C CNN
+F 1 "+5V" H 5415 4223 50  0000 C CNN
 F 2 "" H 5400 4050 50  0001 C CNN
 F 3 "" H 5400 4050 50  0001 C CNN
 	1    5400 4050
-	-1   0    0    1
-$EndComp
-$Comp
-L power:GND #PWR0104
-U 1 1 616F03D4
+	1    0    0    -1
+$EndComp
+$Comp
+L power:+5V #PWR0104
+U 1 1 61A8246D
 P 6100 4050
-F 0 "#PWR0104" H 6100 3800 50  0001 C CNN
-F 1 "GND" H 6100 3900 50  0000 C CNN
+F 0 "#PWR0104" H 6100 3900 50  0001 C CNN
+F 1 "+5V" H 6115 4223 50  0000 C CNN
 F 2 "" H 6100 4050 50  0001 C CNN
 F 3 "" H 6100 4050 50  0001 C CNN
 	1    6100 4050
-	-1   0    0    1
-$EndComp
-$Comp
-L power:GND #PWR0108
-U 1 1 616F0AF2
+	1    0    0    -1
+$EndComp
+$Comp
+L power:+5V #PWR0108
+U 1 1 61A828CA
 P 6900 4050
-F 0 "#PWR0108" H 6900 3800 50  0001 C CNN
-F 1 "GND" H 6900 3900 50  0000 C CNN
+F 0 "#PWR0108" H 6900 3900 50  0001 C CNN
+F 1 "+5V" H 6915 4223 50  0000 C CNN
 F 2 "" H 6900 4050 50  0001 C CNN
 F 3 "" H 6900 4050 50  0001 C CNN
 	1    6900 4050
-	-1   0    0    1
-$EndComp
-$Comp
-L power:+5V #PWR0109
-U 1 1 616F248F
-P 4800 4850
-F 0 "#PWR0109" H 4800 4700 50  0001 C CNN
-F 1 "+5V" H 4815 5023 50  0000 C CNN
-F 2 "" H 4800 4850 50  0001 C CNN
-F 3 "" H 4800 4850 50  0001 C CNN
-	1    4800 4850
-	-1   0    0    1
-$EndComp
-$Comp
-L power:+5V #PWR0110
-U 1 1 616F30CA
-P 5550 4850
-F 0 "#PWR0110" H 5550 4700 50  0001 C CNN
-F 1 "+5V" H 5565 5023 50  0000 C CNN
-F 2 "" H 5550 4850 50  0001 C CNN
-F 3 "" H 5550 4850 50  0001 C CNN
-	1    5550 4850
-	-1   0    0    1
-$EndComp
-$Comp
-L power:+5V #PWR0111
-U 1 1 616F3611
-P 6300 4850
-F 0 "#PWR0111" H 6300 4700 50  0001 C CNN
-F 1 "+5V" H 6315 5023 50  0000 C CNN
-F 2 "" H 6300 4850 50  0001 C CNN
-F 3 "" H 6300 4850 50  0001 C CNN
-	1    6300 4850
-	-1   0    0    1
-$EndComp
-Wire Wire Line
-	5400 4600 5400 4500
-Wire Wire Line
-	6000 4150 5400 4150
-Wire Wire Line
-	5400 4150 5400 4200
-Wire Wire Line
-	6100 4200 6100 4150
-Wire Wire Line
-	6100 4500 6100 4600
-Wire Wire Line
-	6000 3150 6000 4150
-Wire Wire Line
-	6100 4150 6100 4050
-Connection ~ 6100 4150
-Wire Wire Line
-	6200 4150 6200 3150
-Wire Wire Line
-	6900 4600 6900 4500
-Wire Wire Line
-	6900 4200 6900 4150
-Connection ~ 6900 4150
-Wire Wire Line
-	6900 4150 6900 4050
-Wire Wire Line
-	6400 4150 6400 3150
-Wire Wire Line
-	5400 4150 5400 4050
-Connection ~ 5400 4150
+	1    0    0    -1
+$EndComp
+$Comp
+L power:GND #PWR?
+U 1 1 61A852F1
+P 4800 5000
+F 0 "#PWR?" H 4800 4750 50  0001 C CNN
+F 1 "GND" H 4805 4827 50  0000 C CNN
+F 2 "" H 4800 5000 50  0001 C CNN
+F 3 "" H 4800 5000 50  0001 C CNN
+	1    4800 5000
+	1    0    0    -1
+$EndComp
+$Comp
+L power:GND #PWR?
+U 1 1 61A85A9B
+P 5550 5000
+F 0 "#PWR?" H 5550 4750 50  0001 C CNN
+F 1 "GND" H 5555 4827 50  0000 C CNN
+F 2 "" H 5550 5000 50  0001 C CNN
+F 3 "" H 5550 5000 50  0001 C CNN
+	1    5550 5000
+	1    0    0    -1
+$EndComp
+$Comp
+L power:GND #PWR?
+U 1 1 61A85E47
+P 6300 5000
+F 0 "#PWR?" H 6300 4750 50  0001 C CNN
+F 1 "GND" H 6305 4827 50  0000 C CNN
+F 2 "" H 6300 5000 50  0001 C CNN
+F 3 "" H 6300 5000 50  0001 C CNN
+	1    6300 5000
+	1    0    0    -1
+$EndComp
+Wire Wire Line
+	4800 4900 4800 5000
+Wire Wire Line
+	5550 4900 5550 5000
+Wire Wire Line
+	6300 4900 6300 5000
 $EndSCHEMATC
